File: TDA2030/TDA2030.kicad_sch (KiCad schematic)
At the start: 18 parts, among them J1 HP 42, J2 In, U1 TDA2030

Commit message: Assing footprint
Parts:
- removed J2: In, symbol Connector:Screw_Terminal_01x02
- added J1: AudioJack2_Ground, Connector_Audio:Jack_3.5mm_CUI_SJ1-3523N_Horizontal, symbol Connector_Audio:AudioJack2_Ground
- added J2: Barrel_Jack, Connector_BarrelJack:BarrelJack_SwitchcraftConxall_RAPC10U_Horizontal, symbol Connector:Barrel_Jack
- added SW1: Power, Button_Switch_THT:SW_PUSH_1P1T_6x3.5mm_H4.3_APEM_MJTP1243, symbol Switch:SW_SPST
- C1: renamed from C3; footprint (none) -> Capacitor_THT:CP_Radial_D5.0mm_P2.50mm
- C2: renamed from C4; footprint (none) -> Capacitor_THT:C_Disc_D11.0mm_W5.0mm_P7.50mm
- C3: renamed from C5; footprint (none) -> Capacitor_THT:CP_Radial_D5.0mm_P2.50mm
- C4: renamed from C6; footprint (none) -> Capacitor_THT:CP_Radial_D5.0mm_P2.00mm
- C5: renamed from C1; footprint (none) -> Capacitor_THT:C_Disc_D5.0mm_W2.5mm_P2.50mm
- C6: renamed from C2; footprint (none) -> Capacitor_THT:CP_Radial_D10.0mm_P7.50mm
- J3: renamed from J1; footprint (none) -> TerminalBlock_Phoenix:TerminalBlock_Phoenix_MKDS-1,5-2-5.08_1x02_P5.08mm_Horizontal
- R1: renamed from R2; footprint (none) -> PCM_Resistor_THT_AKL:R_Axial_DIN0309_L9.0mm_D3.2mm_P15.24mm_Horizontal
- R2: renamed from R4; footprint (none) -> PCM_Resistor_THT_AKL:R_Axial_DIN0309_L9.0mm_D3.2mm_P15.24mm_Horizontal
- R3: footprint (none) -> PCM_Resistor_THT_AKL:R_Axial_DIN0309_L9.0mm_D3.2mm_P15.24mm_Horizontal
- R4: renamed from R5; footprint (none) -> PCM_Resistor_THT_AKL:R_Axial_DIN0309_L9.0mm_D3.2mm_P15.24mm_Horizontal
- R5: renamed from R6; footprint (none) -> PCM_Resistor_THT_AKL:R_Axial_DIN0309_L9.0mm_D3.2mm_P15.24mm_Horizontal
- R6: renamed from R1; footprint (none) -> PCM_Resistor_THT_AKL:R_Axial_DIN0309_L9.0mm_D3.2mm_P15.24mm_Horizontal
- RV1: footprint (none) -> PCM_Potentiometer_THT_AKL:Potentiometer_Piher_T-16H_Single_Horizontal
Connections:
- net GNDREF: now also J1.G, J2.2
- net VCC: now also SW1.1 (A)
- net at RV1.1: now also J1.S
- new net: J2.1, SW1.2 (B)
- no-connect marks 0 -> 1
