File: TDA2030/TDA2030.kicad_pcb (KiCad board)
At the start: 2 copper layers, 75.7 x 58.2 mm, 20 parts, among them J1 AudioJack2_Ground, J2 Barrel_Jack, J3 HP 42, SW1 Power, U1 TDA2030

Commit message: Routing PCB
Parts:
- moved R6 166.5 mm to (141.6, 56.0), turned to 180 degrees
- moved J3 148.6 mm to (141.7, 37.3), turned to 180 degrees
- moved C3 137.3 mm to (112.4, 54.0), turned to 90 degrees
- moved C1 137.2 mm to (112.0, 45.0), turned to 90 degrees
- moved R5 136.1 mm to (110.1, 67.0)
- moved D2 133.6 mm to (115.6, 73.9), turned to -90 degrees
- moved R4 133.1 mm to (106.6, 66.3), turned to -90 degrees
- moved R2 132.2 mm to (105.8, 55.7), turned to 90 degrees
- moved D1 130.0 mm to (111.5, 81.5), turned to 90 degrees
- moved R3 126.4 mm to (100.6, 55.7), turned to 90 degrees
- moved C4 126.3 mm to (102.1, 79.9), turned to 180 degrees
- moved C5 122.2 mm to (126.8, 46.4), turned to 90 degrees
- moved R1 119.7 mm to (94.5, 40.5), turned to -90 degrees
- moved C6 114.6 mm to (135.7, 48.3)
- moved C2 112.0 mm to (118.2, 50.3), turned to 90 degrees
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Routing:
- net GNDREF: track 0.00 -> 173.2 mm
- net VCC: track 0.00 -> 136.7 mm
- net V+: track 0.00 -> 117.9 mm
- net Net-(D1-A): track 0.00 -> 59.1 mm
- net Net-(J1-PadS): track 0.00 -> 58.2 mm
- net Net-(U1--): track 0.00 -> 56.1 mm
- net Net-(SW1-B): track 0.00 -> 30.4 mm
- net Net-(C3-Pad1): track 0.00 -> 18.6 mm
- net Net-(J3-Pin_1): track 0.00 -> 11.7 mm
- net Net-(C5-Pad1): track 0.00 -> 9.77 mm
- net Net-(C4-Pad1): track 0.00 -> 5.33 mm
- added copper zone on B.Cu, net GNDREF
Other:
- board size 75.7 x 58.2 mm -> 81.5 x 57.2 mm

Commit message: Adding vias for fixation
Routing:
- net GNDREF: vias 0 -> 4
Other:
- outline, holes or cut-outs redrawn
Changed lines of the file:
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@@
 		)
 	)
-	(gr_rect
-		(start 72.5 31)
-		(end 154 88.25)
+	(gr_arc
+		(start 75.5 88.25)
+		(mid 73.37868 87.37132)
+		(end 72.5 85.25)
 		(stroke
 			(width 0.05)
 			(type default)
 		)
-		(fill none)
+		(layer "Edge.Cuts")
+	)
+	(gr_arc
+		(start 154 85.25)
+		(mid 153.12132 87.37132)
+		(end 151 88.25)
+		(stroke
+			(width 0.05)
+			(type default)
+		)
+		(layer "Edge.Cuts")
+	)
+	(gr_line
+		(start 154 34)
+		(end 154 85.25)
+		(stroke
+			(width 0.05)
+			(type default)
+		)
+		(layer "Edge.Cuts")
+	)
+	(gr_arc
+		(start 72.5 34)
+		(mid 73.37868 31.87868)
+		(end 75.5 31)
+		(stroke
+			(width 0.05)
+			(type default)
+		)
+		(layer "Edge.Cuts")
+	)
+	(gr_line
+		(start 151 88.25)
+		(end 75.5 88.25)
+		(stroke
+			(width 0.05)
+			(type default)
+		)
+		(layer "Edge.Cuts")
+	)
+	(gr_arc
+		(start 151 31)
+		(mid 153.12132 31.87868)
+		(end 154 34)
+		(stroke
+			(width 0.05)
+			(type default)
+		)
+		(layer "Edge.Cuts")
+	)
+	(gr_line
+		(start 75.5 31)
+		(end 151 31)
+		(stroke
+			(width 0.05)
+			(type default)
+		)
+		(layer "Edge.Cuts")
+	)
+	(gr_line
+		(start 72.5 85.25)
+		(end 72.5 34)
+		(stroke
+			(width 0.05)
+			(type default)
+		)
 		(layer "Edge.Cuts")
 	)
@@
 		(layer "User.4")
 	)
+	(via
+		(at 150 34.4)
+		(size 4)
+		(drill 3)
+		(layers "F.Cu" "B.Cu")
+		(free yes)
+		(net 1)
+	)
+	(via
+		(at 75.4 35.2)
+		(size 4)
+		(drill 3)
+		(layers "F.Cu" "B.Cu")
+		(free yes)
+		(net 1)
+	)
+	(via
+		(at 76 84.2)
+		(size 4)
+		(drill 3)
+		(layers "F.Cu" "B.Cu")
+		(free yes)
+		(net 1)
+	)
+	(via
+		(at 149.2 83.6)
+		(size 4)
+		(drill 3)
+		(layers "F.Cu" "B.Cu")
+		(free yes)
+		(net 1)
+	)
 	(segment
